File: PCB/unimodule.sch (EAGLE design)
At the start: 130 parts, among them IC1 TTGO_DISP, IC2 DS18D20, IC3 FAN3111E, IC4 FAN3111E, IC5 FAN3111E, K1 XY2500(5.0)-4PV, K100 JSM1-12V-5, K101 XY2500(5.0)-4PV, K102 JST-B02B-JWPF-SK-R, K103 JST-B04B-JWPF-SK-R, K104 JST-B08B-JWPF-SK-R, K105 JST-B03B-JWPF-SK-R, U1 MAX3485, U2 LMR62014XMFE/NOPB0

Commit message: almost ready
Parts:
- added C25: 22uF, rcl:C-EUC1206
- added SJ1: (no value), siliXcon-pads:SMD-JUMPER
- R9: device rcl:R-EU_0204/7 -> rcl:R-EU_0207/10
Connections:
- removed net DO1: IC3.IN
- net +10V: now also SJ1.2
- net +3V3: now also C25.1
- net +5V: now also SJ1.1
- net DO_1: now also IC3.IN
- net GND: now also C25.2
Other:
- moved on the sheet: C10, C11, C12, C13, C24, D3, IC3, IC4, IC5, K101, L1, R14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

Commit message: Fix components height
Parts:
- D3: device diode:DIODE-SOD323-W -> siliXcon-semiconductors:PMEG4005EH
- OK1, OK2, OK3: device optocoupler:MOC3023M -> siliXcon-ICs:MOC30
Changed lines of the file:
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@@
 </classes>
 <parts>
-<part name="OK3" library="optocoupler" library_urn="urn:adsk.eagle:library:320" deviceset="MOC30*M" device="" package3d_urn="urn:adsk.eagle:package:21942/1" technology="23" value="MOC3063M"/>
+<part name="OK3" library="siliXcon-ICs" deviceset="MOC30" device="" value="MOC3063M"/>
 <part name="OK4" library="optocoupler" library_urn="urn:adsk.eagle:library:320" deviceset="4N35" device="" package3d_urn="urn:adsk.eagle:package:21942/1"/>
 <part name="D2" library="diode" library_urn="urn:adsk.eagle:library:210" deviceset="1N4004" device="" package3d_urn="urn:adsk.eagle:package:43336/1"/>
@@
 <part name="GND4" library="siliXcon-supply" deviceset="GND" device=""/>
 <part name="R106" library="rcl" library_urn="urn:adsk.eagle:library:334" deviceset="R-EU_" device="R0603" package3d_urn="urn:adsk.eagle:package:23555/3" value="220R"/>
-<part name="OK2" library="optocoupler" library_urn="urn:adsk.eagle:library:320" deviceset="MOC30*M" device="" package3d_urn="urn:adsk.eagle:package:21942/1" technology="23" value="MOC3063M"/>
+<part name="OK2" library="siliXcon-ICs" deviceset="MOC30" device="" value="MOC3063M"/>
 <part name="U$3" library="siliXcon-semiconductors" deviceset="BT139B" device="" value="BT139B-600E"/>
 <part name="R104" library="rcl" library_urn="urn:adsk.eagle:library:334" deviceset="R-EU_" device="R1206" package3d_urn="urn:adsk.eagle:package:23540/2" value="380R"/>
@@
 <part name="GND5" library="siliXcon-supply" deviceset="GND" device=""/>
 <part name="R105" library="rcl" library_urn="urn:adsk.eagle:library:334" deviceset="R-EU_" device="R0603" package3d_urn="urn:adsk.eagle:package:23555/3" value="220R"/>
-<part name="OK1" library="optocoupler" library_urn="urn:adsk.eagle:library:320" deviceset="MOC30*M" device="" package3d_urn="urn:adsk.eagle:package:21942/1" technology="23" value="MOC3063M"/>
+<part name="OK1" library="siliXcon-ICs" deviceset="MOC30" device="" value="MOC3063M"/>
 <part name="U$2" library="siliXcon-semiconductors" deviceset="BT139B" device="" value="BT139B-600E"/>
 <part name="R6" library="rcl" library_urn="urn:adsk.eagle:library:334" deviceset="R-EU_" device="R1206" package3d_urn="urn:adsk.eagle:package:23540/2" value="380R"/>
@@
 </part>
 <part name="U2" library="siliXcon-ICs" deviceset="LMR62014XMFE/NOPB" device="0"/>
-<part name="D3" library="diode" deviceset="DIODE-" device="SOD323-W" value="PMEG4005AEA"/>
-<part name="C10" library="rcl" deviceset="C-EU" device="C1206" value="22uF"/>
-<part name="C11" library="rcl" deviceset="C-EU" device="C1206" value="22uF"/>
+<part name="D3" library="siliXcon-semiconductors" deviceset="PMEG4005" device="EH" value="PMEG4005AEA"/>
+<part name="C10" library="rcl" library_urn="urn:adsk.eagle:library:334" deviceset="C-EU" device="C1206" package3d_urn="urn:adsk.eagle:package:23618/2" value="22uF"/>
+<part name="C11" library="rcl" library_urn="urn:adsk.eagle:library:334" deviceset="C-EU" device="C1206" package3d_urn="urn:adsk.eagle:package:23618/2" value="22uF"/>
 <part name="GND23" library="supply1" library_urn="urn:adsk.eagle:library:371" deviceset="GND" device=""/>
 <part name="GND24" library="supply1" library_urn="urn:adsk.eagle:library:371" deviceset="GND" device=""/>
-<part name="R15" library="rcl" deviceset="R-EU_" device="R0603" value="6k8"/>
-<part name="R16" library="rcl" deviceset="R-EU_" device="R0603" value="47k"/>
+<part name="R15" library="rcl" library_urn="urn:adsk.eagle:library:334" deviceset="R-EU_" device="R0603" package3d_urn="urn:adsk.eagle:package:23555/3" value="6k8"/>
+<part name="R16" library="rcl" library_urn="urn:adsk.eagle:library:334" deviceset="R-EU_" device="R0603" package3d_urn="urn:adsk.eagle:package:23555/3" value="47k"/>
 <part name="GND25" library="supply1" library_urn="urn:adsk.eagle:library:371" deviceset="GND" device=""/>
-<part name="C12" library="rcl" deviceset="C-EU" device="C0603" value="270p"/>
+<part name="C12" library="rcl" library_urn="urn:adsk.eagle:library:334" deviceset="C-EU" device="C0603" package3d_urn="urn:adsk.eagle:package:23616/2" value="270p"/>
 <part name="GND26" library="supply1" library_urn="urn:adsk.eagle:library:371" deviceset="GND" device=""/>
 <part name="L1" library="rcl" deviceset="L-US" device="" value="1206F-100K-01, ILSB1206ER100K"/>

Commit message: add connector description
Connections:
- net N$16 renamed R_NO
- net N$17 renamed R_C
- net N$18 renamed R_NC
- net N$22 renamed SDA_P
- net N$29 renamed SCL_P
- net N$30 renamed PWM_2
- net N$32 renamed PWM_1
- net N$35 renamed PWM_3
Changed lines of the file:
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@@
 </segment>
 </net>
-<net name="N$16" class="1">
+<net name="R_NO" class="1">
 <segment>
 <pinref part="U$100" gate="G$1" pin="3"/>
@@
 <pinref part="K100" gate="G$1" pin="3"/>
 <wire x1="228.6" y1="88.9" x2="228.6" y2="83.82" width="0.1524" layer="91"/>
-</segment>
-</net>
-<net name="N$17" class="1">
+<label x="203.2" y="88.9" size="1.778" layer="95" rot="R180" xref="yes"/>
+</segment>
+</net>
+<net name="R_C" class="1">
 <segment>
 <pinref part="K100" gate="G$1" pin="1"/>
@@
 </segment>
 </net>
-<net name="N$18" class="0">
+<net name="R_NC" class="0">
 <segment>
 <pinref part="U$100" gate="G$1" pin="1"/>
@@
 <wire x1="203.2" y1="60.96" x2="228.6" y2="60.96" width="0.1524" layer="91"/>
 <wire x1="228.6" y1="60.96" x2="228.6" y2="63.5" width="0.1524" layer="91"/>
+<label x="203.2" y="60.96" size="1.778" layer="95" rot="R180" xref="yes"/>
 </segment>
 </net>
@@
 </segment>
 </net>
-<net name="N$22" class="0">
+<net name="SDA_P" class="0">
 <segment>
 <pinref part="K103" gate="G$1" pin="3"/>
@@
 </segment>
 </net>
-<net name="N$29" class="0">
+<net name="SCL_P" class="0">
 <segment>
 <pinref part="R13" gate="G$1" pin="2"/>
@@
 </segment>
 </net>
-<net name="N$32" class="0">
+<net name="PWM_1" class="0">
 <segment>
 <pinref part="R14" gate="G$1" pin="2"/>
@@
 </segment>
 </net>
-<net name="N$30" class="0">
+<net name="PWM_2" class="0">
 <segment>
 <pinref part="R17" gate="G$1" pin="2"/>
@@
 </segment>
 </net>
-<net name="N$35" class="0">
+<net name="PWM_3" class="0">
 <segment>
 <pinref part="R18" gate="G$1" pin="2"/>

Commit message: add status LEDs
Parts:
- added C26: DISP_BATSMD, TTGO_LCD_DISP:DISP_BATSMD
- added C27: DISP_BAT2,54, TTGO_LCD_DISP:DISP_BAT2,54
- added LED10, LED11, LED12, LED13, LED14, LED7, LED8, LED9: (no value), siliXcon-semiconductors:LED0603
- added R39, R40, R41, R42, R43: 220R, rcl:R-EU_R0603
- added R44, R45, R46: 1k, rcl:R-EU_R0603
- C100: value 220uF / 6.3V -> 330uF / 6.3V; device rcl:CPOL-EUE2.5-6 -> rcl:CPOL-EUE2.5-7
- C101: value 220uF / 6.3V -> 330uF / 6.3V
- K100: value JSM1-12V-5 -> G5LE-1-E 5VDC OMRON
Connections:
- new net BAT+: C26.BAT+, C27.BAT+
- new net BAT-: C26.BAT-, C27.BAT-
- new net N$16: LED7.A, R39.2
- new net N$17: LED8.A, R40.2
- new net N$18: LED9.A, R41.2
- new net N$21: LED10.A, R42.2
- new net N$22: LED11.A, R43.2
- new net N$29: LED12.A, R44.2
- new net N$30: LED13.A, R45.2
- new net N$32: LED14.A, R46.2
- net +3V3: now also R43.1
- net GND: now also LED10.C, LED11.C, LED12.C, LED13.C, LED14.C, LED7.C, LED8.C, LED9.C
- net OUT_1_SIG: now also R39.1
- net OUT_2_SIG: now also R40.1
- net OUT_3_SIG: now also R41.1
- net PWM_1: now also R44.1
- net PWM_2: now also R45.1
- net PWM_3: now also R46.1
- net RELAY_SIG: now also R42.1

Commit message: silk screen organize
Parts:
- removed C22, C23: 100n, rcl:C-EUC0603
- removed C25: 22uF, rcl:C-EUC1206
- removed C26: DISP_BATSMD, TTGO_LCD_DISP:DISP_BATSMD
- removed FD4: (no value), siliXcon-pads:FIDUCIAL-MARKER2MM
- removed K1: XY2500(5.0)-4PV, siliXcon-connectors:XY2500(5.0)-4PV
- removed R38: 10k, rcl:R-EU_R0603
- removed R39, R40, R41, R42, R43: 220R, rcl:R-EU_R0603
- removed R44, R45, R46: 1k, rcl:R-EU_R0603
- removed SJ1: (no value), siliXcon-pads:SMD-JUMPER
- removed U$11: BAT54SFILM, siliXcon-semiconductors:BAT54SFILM
- added C102, C103, C106: 100n, rcl:C-EUC0603
- added C105: 22uF, rcl:C-EUC1206
- added FD100: (no value), siliXcon-pads:FIDUCIAL-MARKER2MM
- added K106: JST-B03B-JWPF-SK-R, siliXcon-connectors:JST-B03B-JWPF-SK-R
- added R109, R110, R111: 1k, rcl:R-EU_R1206
- added R112, R113, R114, R115, R116, R117: 10k, rcl:R-EU_R0603
- added SJ101: (no value), siliXcon-pads:NET-TIE
- added U$105: IRM-03-05, siliXcon-modules:IRM-03
- C1: value (none) -> 100n
- C10, C5, C6: value 22uF -> 100n; device rcl:C-EUC1206 -> rcl:C-EUC0603
- C11: value 22uF -> DISP_BATSMD; device rcl:C-EUC1206 -> TTGO_LCD_DISP:DISP_BATSMD
- C13, C14, C19, C20, C4: value 100n -> 22uF; device rcl:C-EUC0603 -> rcl:C-EUC1206
- C2: value 22uF -> !DNP 100n; device rcl:C-EUC1206 -> rcl:C-EUC0603
- C3: value 100n -> (none)
- C7: value !DNP 100n -> 100n
- D1: value (none) -> PMEG4005AEA
- D2: value 1N4004 -> (none); device diode:1N4004 -> siliXcon-semiconductors:PMEG4005EH
- D3: value PMEG4005AEA -> 1N4004; device siliXcon-semiconductors:PMEG4005EH -> diode:1N4004
- K102: value JST-B02B-JWPF-SK-R -> XY2500(5.0)-4PV; device siliXcon-connectors:JST-B02B-JWPF-SK-R -> siliXcon-connectors:XY2500(5.0)-4PV
- K103: value JST-B04B-JWPF-SK-R -> JST-B08B-JWPF-SK-R; device siliXcon-connectors:JST-B04B-JWPF-SK-R -> siliXcon-connectors:JST-B08B-JWPF-SK-R
- K104: value JST-B08B-JWPF-SK-R -> JST-B04B-JWPF-SK-R; device siliXcon-connectors:JST-B08B-JWPF-SK-R -> siliXcon-connectors:JST-B04B-JWPF-SK-R
- K105: value JST-B03B-JWPF-SK-R -> JST-B02B-JWPF-SK-R; device siliXcon-connectors:JST-B03B-JWPF-SK-R -> siliXcon-connectors:JST-B02B-JWPF-SK-R
- LED14: value (none) -> WS2812B5050; device siliXcon-semiconductors:LED0603 -> adafruit:WS2812B5050
- LED4: value WS2812B5050 -> (none); device adafruit:WS2812B5050 -> siliXcon-semiconductors:LED0603
- R10, R9: value 30k -> (none); device rcl:R-EU_0207/10 -> rcl:R-EU_R0603
- R105: value 220R -> 380R; device rcl:R-EU_R0603 -> rcl:R-EU_R1206
- R108: value (none) -> 220R
- R11, R12, R5: value 4k7 -> 100R
- R14: value 1k -> 220R; device rcl:R-EU_R1206 -> rcl:R-EU_R0603
- R15: value 6k8 -> 10k
- R16: value 47k -> 10k
- R17: value 1k -> 10k; device rcl:R-EU_R1206 -> rcl:R-EU_R0603
- R18: value 1k -> 6k8; device rcl:R-EU_R1206 -> rcl:R-EU_R0603
- R19: value (none) -> 10k
- R20: value 100R -> 10k
- R23: value 10k -> 100R
- R25: value 10k -> 47k
- R26, R29: value 100R -> 1k
- R27, R28: value 10k -> 1k
- R3: value 1k -> 4k7
- R30, R31, R33: value 10k -> 220R
- R32: value 100R -> 220R
- R34: value 10k -> 100k
- R35: value 100R -> 100k
- R36, R37: value 10k -> 30k; device rcl:R-EU_R0603 -> rcl:R-EU_0207/10
- R4: value 100k -> 100R
- R6: value 380R -> 100R; device rcl:R-EU_R1206 -> rcl:R-EU_R0603
- R7: value 100k -> 4k7
- R8: value 100R -> 4k7
- SJ100: device siliXcon-pads:NET-TIE -> siliXcon-pads:SMD-JUMPER
- U$1: value IRM-03-05 -> BAT54SFILM; device siliXcon-modules:IRM-03 -> siliXcon-semiconductors:BAT54SFILM
- U$10, U$8, U$9: value BAT54SFILM -> BT139B-600E; device siliXcon-semiconductors:BAT54SFILM -> siliXcon-semiconductors:BT139B
- U$2, U$3, U$4: value BT139B-600E -> BAT54SFILM; device siliXcon-semiconductors:BT139B -> siliXcon-semiconductors:BAT54SFILM
- renumbered C24 to C104, C27 to C107, FD3 to FD101, IC2 to IC103, IC3 to IC100, IC4 to IC101, IC5 to IC102
Connections:
- removed net N$27 (its old number): LED4.DO, LED5.DI
- new net N$28: LED14.DI, LED6.DO
- net +10V: now also C103.2, C14.1, D1.C, R25.1, SJ100.2; no longer C11.1, C13.2, D3.C, R16.1, SJ1.2
- net +3V3: now also C1.2, C10.1, C102.2, C106.1, C15.2, K103.8, K104.4, K106.3, R115.1, R116.1, R117.1, R14.1, R19.1, R20.1, R29.2, R7.2, R8.2, R9.2, U$1.C, U$2.C, U$3.C, U$4.C; no longer C14.1, C21.2, C22.2, C23.2, C25.1, K103.4, K104.8, K105.3, R108.2, R11.2, R12.2, R25.1, R28.1, R31.1, R34.1, R37.1, R43.1, R5.2, U$10.C, U$11.C, U$8.C, U$9.C
- net +5V: now also C105.1, C13.1, C19.1, C20.1, D2.C, LED14.VDD, SJ100.1, U$105.V+; no longer C10.1, C2.1, C5.1, C6.1, D1.C, LED4.VDD, SJ1.1, U$1.V+
- net A1: now also K102.4, K103.1, R15.1, R19.2, R24.1; no longer K1.4, K104.1, R35.1, R37.2, R38.1
- net A2: now also K102.3, K103.2, R16.1, R20.2, R23.1; no longer K1.3, K104.2, R29.1, R31.2, R33.1
- net A3: now also K102.2, K103.3, R17.1, R21.2, R22.1; no longer K1.2, K104.3, R32.1, R34.2, R36.1
- net A4: now also K103.5, R11.1, R114.1, R117.2; no longer K104.5, R21.2, R22.1, R23.1
- net A5: now also K103.6, R113.1, R116.2, R12.1; no longer K104.6, R26.1, R28.2, R30.1
- net A6: now also K103.7, R112.1, R115.2, R13.1; no longer K104.7, R24.1, R25.2, R27.1
- net AIN_1: now also C18.1, R24.2, U$7.COMMON; no longer C20.1, R35.2, U$5.COMMON
- net AIN_2: now also C17.1, R23.2; no longer C18.1, R29.2
- net AIN_3: now also C16.1, R22.2, U$5.COMMON; no longer C19.1, R32.2, U$7.COMMON
- net AIN_4: now also C5.1, R11.2, U$2.COMMON; no longer C15.1, R22.2, U$10.COMMON
- net AIN_5/DO_2: now also C6.1, R12.2, U$3.COMMON; no longer C17.1, R26.2, U$9.COMMON
- net AIN_6/DO_3: now also C7.1, R13.2, U$4.COMMON; no longer C16.1, R24.2, U$8.COMMON
- net BAT+: now also C11.BAT+; no longer C26.BAT+
- net BAT-: now also C11.BAT-; no longer C26.BAT-
- net DALAS_TEMP: now also K106.2, R3.1, U$1.COMMON; no longer K105.2, R5.1, U$11.COMMON
- net ENC: now also C3.1, R1.1; no longer C1.1, R19.1
- net ENC_2: now also K105.2, R10.2, R9.1, SJ101.2; no longer K102.2, R108.1, R19.2, SJ100.2
- net GND: now also C1.1, C102.1, C103.1, C105.2, C106.2, C13.2, C15.1, C21.2, K103.4, K104.1, K106.1, LED14.GND, LED4.C, R112.2, R113.2, R114.2, R15.2, R16.2, R17.2, R18.1, R34.2, R5.2, U$1.A, U$105.V-, U$2.A, U$3.A, U$4.A; no longer C1.2, C11.2, C13.1, C15.2, C21.1, C22.1, C23.1, C25.2, K1.1, K103.1, K104.4, LED14.C, LED4.GND, R15.1, R20.2, R23.2, R27.2, R30.2, R33.2, R36.2, R38.2, R7.2, U$1.V-, U$10.A, U$11.A, U$8.A, U$9.A
- net L_FUSED: now also R105.1, U$10.A2, U$8.A2, U$9.A2; no longer R6.1, U$2.A2, U$3.A2, U$4.A2
- net L_IN: now also U$105.AC/L; no longer U$1.AC/L
- net L_OUT_1: now also R100.2, U$9.A1; no longer R102.2, U$2.A1
- net L_OUT_2: now also U$8.A1; no longer U$3.A1
- net L_OUT_3: now also R102.2, U$10.A1; no longer R100.2, U$4.A1
- net N: now also R37.2, U$105.AC/N; no longer R9.2, U$1.AC/N
- net N$1: now also D3.A; no longer D2.A
- net N$10: now also R107.2; no longer R105.2
- net N$11: now also R104.2; no longer R6.2
- net N$12: now also R100.1, U$9.G; no longer R102.1, U$2.G
- net N$13: now also R106.2; no longer R107.2
- net N$14: now also R10.1; no longer R2.1
- net N$15: now also SJ101.1; no longer SJ100.1
- net N$16: now also LED10.A, R30.2; no longer LED7.A, R39.2
- net N$17: now also LED11.A, R31.2; no longer LED8.A, R40.2
- net N$18: now also LED12.A, R32.2; no longer LED9.A, R41.2
- net N$2: now also D3.C, R36.1; no longer D2.C, R10.1
- net N$20: now also D2.A; no longer D1.A
- net N$21: now also LED13.A, R33.2; no longer LED10.A, R42.2
- net N$22: now also LED4.A, R14.2; no longer LED11.A, R43.2
- net N$23: now also R110.1; no longer R17.1
- net N$24: now also D1.A; no longer D3.A
- net N$26: now also LED5.DI; no longer LED4.DI
- net N$29: now also LED9.A, R28.2; no longer LED12.A, R44.2
- net N$3: now also R2.1; no longer R1.1
- net N$30: now also LED8.A, R27.2; no longer LED13.A, R45.2
- net N$31: now also R109.1; no longer R14.1
- net N$32: now also LED7.A, R26.2; no longer LED14.A, R46.2
- net N$33: now also R111.1; no longer R18.1
- net N$34: now also R18.2, R25.2; no longer R15.2, R16.2
- net N$38: now also R5.1; no longer R20.1
- net N$4: now also R37.1; no longer R9.1
- net N$5: now also R105.2; no longer R103.2
- net N$6: now also R102.1, U$10.G; no longer R100.1, U$4.G
- net N$7: now also R103.2; no longer R104.2
- net N$8: now also R108.2; no longer R106.2
- net N$9: now also U$8.G; no longer U$3.G
- net OUT_1_SIG: now also R106.1, R30.1; no longer R107.1, R39.1
- net OUT_2_SIG: now also R107.1, R31.1; no longer R105.1, R40.1
- net OUT_3_SIG: now also R108.1, R32.1; no longer R106.1, R41.1
- net PWM_1: now also R109.2, R28.1; no longer R14.2, R44.1
- net PWM_2: now also R110.2, R27.1; no longer R17.2, R45.1
- net PWM_3: now also R111.2, R26.1; no longer R18.2, R46.1
- net RELAY_SIG: now also R33.1, R34.1; no longer R42.1, R7.1
- net SCL: now also C2.1, R4.1; no longer C9.1, R13.1
- net SCL_P: now also K104.2, R4.2, R7.1; no longer K103.2, R11.1, R13.2
- net SDA: now also C9.1, R6.1; no longer C7.1, R8.1
- net SDA_P: now also K104.3, R6.2, R8.1; no longer K103.3, R12.1, R8.2
- net SENS_IN: now also R36.2; no longer R10.2
- net ZC: now also R29.1, R35.2; no longer R3.1, R4.2
- net ZC_SIG: now also C21.1, R35.1; no longer C3.1, R4.1
